File: hardware/electronics/testbench/kicad-project/testbench.kicad_sch (KiCad schematic)
At the start: 0 parts

Commit message: added devboards and gitignore
Parts:
- added U1: NUCLEO-G431RB, local:MODULE_NUCLEO-G431RB, symbol NUCLEO-G431RB:NUCLEO-G431RB
- added U2: ESP32-S3-DEVKITC-1-N8R8, local:ESP32-S3-DEVKITC-1-N8R8, symbol ESP32-S3-DEVKITC-1-N8R8:ESP32-S3-DEVKITC-1-N8R8
Connections:
- new net: U1.CN10_10 (NC), U1.CN10_36 (NC), U1.CN10_38 (NC), U1.CN7_10 (NC), U1.CN7_11 (NC), U1.CN7_26 (NC), U1.CN7_9 (NC)
- new net GND: U1.CN10_20 (GND), U1.CN10_9 (GND), U1.CN7_19 (GND), U1.CN7_20 (GND), U1.CN7_22 (GND), U1.CN7_8 (GND)
- new net GND_1: U1.CN5_7 (GND_1), U1.CN6_6 (GND_1), U1.CN6_7 (GND_1)
